File: USB_Dongle_KiCad.kicad_pcb (KiCad board)
At the start: 6 copper layers, 70 x 27 mm, 59 parts, among them J1 USB_C_Receptacle_USB2.0, J2 Conn SWD 02x05, J3 DM3BT-DSF-PEJS, SW1 PCM12SMTR, SW2 KMR223G LFG, U1 AMS1117-3.3, U2 USB3343, U3 USBULC6-2M6, U4 ESDA14V2-2BF3, U5 STM32F730R8Tx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

Commit message: Fix: Value of external capacitor for VCAP1
Parts:
- removed C13: 100n, Capacitor_SMD:C_0603_1608Metric
- C11: value 100n -> 2.2u
- moved C11 1.60 mm to (117.2, 68.9)
Connections:
- J1 pad S1: (no net) -> unconnected-(J1-SHIELD-PadS1)_1
Routing:
- net GND: track 83.7 -> 79.6 mm, vias 48 -> 47
- net Net-(U5-VCAP_1): track 7.14 -> 5.53 mm
